File: board.brd (EAGLE design)
At the start: 39.7 x 39.7 mm, 22 parts, among them J2 TX, J3 TX, J4 TX, J5 TX, J6 TX, J7 TX, J8 TX, U1 AS5047D, U2 ATMEGA328P_TQFP, Y1 20MHz

Commit message: Board v2
Parts:
- added C4: 0.1u, rcl:C0603
- added LED3: (no value), led:SML0805
- LED1, LED2: device led:SML0603 -> led:SML0805
- moved J3 13.7 mm to (25.1, 30.0)
- moved R4 5.36 mm to (11.4, 30.5), turned to 270 degrees
- moved R5 5.33 mm to (14.2, 30.5), turned to 180 degrees
- moved C2 3.39 mm to (21.5, 26.7), turned to 90 degrees
- moved J4 3.34 mm to (22.4, 30.0)
- moved R6 3.06 mm to (18.8, 30.2), turned to 180 degrees
- moved R3 2.64 mm to (23.6, 23.1)
- moved LED1 2.36 mm to (15.7, 27.4), turned to 270 degrees
- moved R2 2.03 mm to (14.0, 25.9)
- moved J2 1.62 mm to (4.83, 25.1)
- moved J5 1.30 mm to (9.14, 29.2)
- moved LED2 1.26 mm to (23.6, 26.5), turned to 270 degrees
- moved C1 1.17 mm to (19.4, 26.7)
- moved R1 1.14 mm to (8.38, 27.2)
- moved U1 1.00 mm to (19.1, 20.6)
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Connections:
- removed net LED: LED1.C, U2.23
- removed net N$3 (its old number): J1.2, R4.1
- new net N$13: R2.1, U2.24
- new net N$14: LED1.C, LED3.A, R2.2
- new net N$15: J1.3, R6.1
- net +5V: now also C4.1, J1.5; no longer J1.1, R2.1
- net GND: now also C4.2, J1.4; no longer J1.5
- net N$11: now also J1.2, R5.1; no longer J1.4, R6.1
- net N$7: now also LED3.C, U2.23; no longer R2.2
- net N$8: now also J1.1, R4.1; no longer J1.3, R5.1
Routing:
- net +5V: track 123.6 -> 86.6 mm
- net N$7: track 1.85 -> 7.20 mm
- net N$5: track 10.8 -> 6.58 mm
- net N$14: track 0.00 -> 4.14 mm
- net LED: track 4.04 -> 0.00 mm
- net N$15: track 0.00 -> 3.58 mm
- net N$4: track 8.75 -> 5.26 mm
- net N$3 (its old number): track 3.37 -> 0.00 mm
- net N$12: track 0.00 -> 2.54 mm
- net N$3: track 11.9 -> 9.50 mm
- net N$13: track 0.00 -> 1.95 mm
- net GND: track 51.2 -> 49.4 mm
- net N$8: track 3.28 -> 4.72 mm
- net MISO: track 9.04 -> 10.4 mm
- net SS: track 9.43 -> 10.8 mm
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Other:
- board text added: "1mm"
- board text added: "AS5047D encoder (c) Xek top layer"
- board text added: "U V W – +"
- board text removed: "top"
