File: board.sch (EAGLE design)
At the start: 22 parts, among them J2 TX, J3 TX, J4 TX, J5 TX, J6 TX, J7 TX, J8 TX, U1 AS5047D, U2 ATMEGA328P_TQFP, Y1 20MHz

Commit message: Board v2
Parts:
- added C4: 0.1u, rcl:C-EUC0603
- added LED3: (no value), led:LEDSML0805
- LED1, LED2: device led:LEDSML0603 -> led:LEDSML0805
Connections:
- removed net LED: LED1.C, U2.PC0(ADC0)
- removed net N$3 (its old number): J1.2, R4.1
- new net N$13: R2.1, U2.PC1(ADC1)
- new net N$14: LED1.C, LED3.A, R2.2
- new net N$15: J1.3, R6.1
- net +5V: now also C4.1, J1.5; no longer J1.1, R2.1
- net GND: now also C4.2, J1.4; no longer J1.5
- net N$11: now also J1.2, R5.1; no longer J1.4, R6.1
- net N$7: now also LED3.C, U2.PC0(ADC0); no longer R2.2
- net N$8: now also J1.1, R4.1; no longer J1.3, R5.1
Other:
- moved on the sheet: LED1, R2, R4, R5, R6
